File: Precharge-Circuit/Precharge-Circuit.kicad_sch (KiCad schematic)
At the start: 65 parts, among them J1 Conn_01x05, J2 19427-0040, J3 XH_2pin_Side, J4 XH_2pin_Side, J5 19427-0040, J6 Conn_01x02, J7 Conn_01x03, K1 AZDC6-2AE-12D, K2 G5Q-1A4_DC12, K3 G5Q-1A4_DC12, Q1 2N7002K-AU, Q2 2N7002K-AU, Q3 2N7002K-AU, Q4 2N7002K-AU, U1 TLP291(GB,SE, U2 TLP291(GB,SE, U3 TL431QDBVR, U4 TL431QDBVR

Commit message: 電圧検知信号のインジケータと出力をMOSFET駆動に変更
Parts:
- added C5: 1000p, Capacitor_SMD:C_1206_3216Metric, symbol Device:C
- added D15, D16, D17, D18: BZT52H-C16, ProjectEV:D_SOD-123F_BZT52H-xxx, symbol ProjectEV:D_BZT52H-C16
- added H1, H2, H3, H4: M3, MountingHole:MountingHole_3.2mm_M3_Pad_Via, symbol Mechanical:MountingHole_Pad
- added Q5, Q6, Q7, Q8: 2N7002K-AU, ProjectEV:Package_SOT-23_2N7002K-AU, symbol ProjectEV:Transistor_2N7002K-AU
- added R30, R31, R35, R38: 10k, symbol Device:R
- added R32, R39, R40, R41, R42, R43: 15k, Resistor_SMD:R_2010_5025Metric, symbol Device:R
- added R33, R34, R36, R37: 1M, symbol Device:R
- added R44: 1M, Resistor_SMD:R_1206_3216Metric, symbol Device:R
- C4: value C -> 1000p; footprint (none) -> Capacitor_SMD:C_1206_3216Metric
- R1, R10, R28, R29, R5: value R -> 10k
- R11: value R -> 1M; footprint (none) -> Resistor_SMD:R_1206_3216Metric
- R12, R13, R14, R15, R16, R17, R18, R19: footprint Resistor_SMD:R_1206_3216Metric -> Resistor_SMD:R_2010_5025Metric
- R2, R4, R6, R9: value R -> 1M
- R20: value R -> 82k
- R21: value R -> 13k
- R22, R23, R24, R25: value R -> 15k; footprint (none) -> Resistor_SMD:R_2010_5025Metric
- R26, R27: value R -> 100k
- R3, R7, R8: value R -> 100
Connections:
- net +12V: now also R26.2, R27.2, R28.1, R29.1, R35.1, R38.1; no longer U1.4 (Collector), U2.4 (Collector)
- net GND: now also U1.3 (Emitter), U2.3 (Emitter), C5.2, D15.2 (A), D16.2 (A), D17.2 (A), D18.2 (A), Q5.2 (S), Q6.2 (S), Q7.2 (S), Q8.2 (S), R33.1, R34.1, R36.1, R37.1, R44.2; no longer R26.1, R27.1
- net TS+: now also R32.2, R39.2; no longer R22.2
- net VoltageDetect_OUT_1: now also Q7.3 (D), R35.2; no longer R26.2, R29.1, U1.3 (Emitter)
- net VoltageDetect_OUT_2: now also Q8.3 (D), R38.2; no longer R27.2, R28.1, U2.3 (Emitter)
- net at D14.2 (A), R29.2: now also Q6.3 (D)
- net at U1.2 (Cathode), U2.1 (Anode), U4.3 (K): now also R30.1, R31.2
- net at U2.2 (Cathode), U3.3 (K): now also R31.1
- net at D12.1 (K), R25.1, U1.1 (Anode): now also R30.2, R43.1
- net at D13.2 (A), R28.2: now also Q5.3 (D)
- new net: R39.1, R40.2
- new net: D16.1 (K), D17.1 (K), Q5.1 (G), Q7.1 (G), R26.1, R33.2, R34.2, U1.4 (Collector)
- new net: D15.1 (K), D18.1 (K), Q6.1 (G), Q8.1 (G), R27.1, R36.2, R37.2, U2.4 (Collector)
- new net: C5.1, H4.1, R44.1
- new net: R40.1, R41.2
- new net: R42.1, R43.2
- new net: R41.1, R42.2
- new net: R22.2, R32.1
- no-connect marks 2 -> 5
Other:
- moved on the sheet: C1, D1, D13, D14, D2, D3, K1, Q1, Q2, R1, R2, R22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

Commit message: コネクタ修正、信号出力をプッシュプルに修正
Parts:
- removed D18: BZT52H-C16, ProjectEV:D_SOD-123F_BZT52H-xxx, symbol ProjectEV:D_BZT52H-C16
- removed J1: Conn_01x05, symbol Connector_Generic:Conn_01x05
- removed J3, J4: XH_2pin_Side, Connector_JST:JST_XH_S2B-XH-A_1x02_P2.50mm_Horizontal, symbol Connector_Generic:Conn_01x02
- removed J6: Conn_01x02, symbol Connector_Generic:Conn_01x02
- removed J7: Conn_01x03, symbol Connector_Generic:Conn_01x03
- removed Q7, Q8: 2N7002K-AU, ProjectEV:Package_SOT-23_2N7002K-AU, symbol ProjectEV:Transistor_2N7002K-AU
- removed R34, R37: 1M, symbol Device:R
- removed R35, R38: 10k, symbol Device:R
- added D18, D22: LED, symbol Device:LED
- added D19: PZ1AH11B-AU, ProjectEV:D_SOD-123HE_PZ1AHxxxB-AU, symbol ProjectEV:D_PZ1AH11B-AU
- added D20, D21: BZT52H-C16, ProjectEV:D_SOD-123F_BZT52H-xxx, symbol ProjectEV:D_BZT52H-C16
- added J1, J3, J4: S2P-VH, ProjectEV:Connector_S2P-VH, symbol ProjectEV:Connector_VH_2pin_Side
- added J6: SM02B-PASS-1-TB, ProjectEV:Connector_SM02B-PASS-1-TB, symbol ProjectEV:Connector_SM02B-PASS-1-TB
- added J7: SM03B-PASS-1-TB, ProjectEV:Connector_SM03B-PASS-1-TB, symbol ProjectEV:Connector_SM03B-PASS-1-TB
- added J8: SM04B-PASS-1-TB, ProjectEV:Connector_SM04B-PASS-1-TB, symbol ProjectEV:Connector_SM04B-PASS-1-TB
- added Q10, Q11, Q7: PJA3439-AU_R1_000A1, ProjectEV:Package_SOT-23_PJA3439-AU_R1_000A1, symbol ProjectEV:Transistor_PJA3439-AU_R1_000A1
- added Q9: DMP3098LQ-7, ProjectEV:Package_SOT-23_DMP3098LQ-7, symbol ProjectEV:Transistor_DMP3098LQ-7
- added R45: 100k, symbol Device:R
- added R46: 10k, symbol Device:R
- C4: value 1000p -> C; footprint Capacitor_SMD:C_1206_3216Metric -> (none)
- R1: value 10k -> 100
- R11: value 1M -> 10k; footprint Resistor_SMD:R_1206_3216Metric -> (none)
- R26, R27: value 100k -> 100
Connections:
- net +12V: now also C4.1, D17.1 (K), R11.1, R33.2, R36.2, D19.1 (K), D20.1 (K), Q11.2 (S), Q7.2 (S), Q9.2 (S); no longer R26.2, R27.2, R28.1, R29.1
- net AIR+_Drive: now also J3.1 (Pin_1)
- net AIR+_EN: now also J8.1 (Pin_1)
- net AIR-_DRIVE: now also J4.1 (Pin_1)
- net AIR-_EN: now also J8.3 (Pin_3)
- net GND: now also D18.1 (K), D22.1 (K), J1.2 (Pin_2), J3.2 (Pin_2), J4.2 (Pin_2), J6.2 (Pin_2), J6.MP1 (MountPin), J6.MP2 (MountPin), J7.3 (Pin_3), J7.MP1 (MountPin), J7.MP2 (MountPin), J8.4 (Pin_4), J8.MP1 (MountPin), J8.MP2 (MountPin), R45.1; no longer D17.2 (A), R11.2, R33.1, R36.1
- net SDN_IN: now also D21.1 (K), J1.1 (Pin_1), Q10.2 (S); no longer C4.1, R1.1, R11.1
- net ~{PCHG_EN}: now also J8.2 (Pin_2)
- net at D2.1 (K), Q2.1 (G), R1.2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: no longer Q1.3 (D)
- net at C1.1, D3.1 (K), Q1.1 (G)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: now also D21.2 (A), Q10.1 (G)
- net at D14.2 (A), R29.2: no longer Q6.3 (D)
- net at D13.2 (A), R28.2: no longer Q5.3 (D)
- new net: D16.1 (K), D20.2 (A), Q11.1 (G), Q5.1 (G), R26.2, R33.1
- new net: D15.1 (K), D17.2 (A), Q6.1 (G), Q7.1 (G), R27.2, R36.1
- new net: D18.2 (A), R11.2
- new net: R26.1, U1.4 (Collector)
- new net: Q1.3 (D), Q10.3 (D), R1.1, R46.1
- new net: R27.1, U2.4 (Collector)
- new net: D19.2 (A), Q9.1 (G), R45.2
- new net: J6.1 (Pin_1), Q9.3 (D)
- new net: D22.2 (A), R46.2
- new net Voltage_Detect_1: J7.1 (Pin_1), Q11.3 (D), Q5.3 (D), R28.1
- new net Voltage_Detect_2: J7.2 (Pin_2), Q6.3 (D), Q7.3 (D), R29.1
Other:
- note added: "HIGH"
- note added: "HV Active (>= 270 V)"
- note added: "HV Active (>= 60 V)"
- note added: "HV Inactive (or No Connection)"
- note added: "LOW"
- note added: "Voltage_Detect_1"
- note added: "Voltage_Detect_2"
- note added: "x"
- moved on the sheet: C5, D10, D11, D13, D14, D15, D16, H1, H2, H3, H4, Q5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

Commit message: アノテーションし直し
Parts:
- C1: renamed from C2; value C -> 0.1u
- C2: renamed from C4; value C -> 10u
- C3: renamed from C1; value C -> 0.1u
- C4: renamed from C3; value C -> 0.1u
- renumbered D19 to D1, D22 to D10, D20 to D11, D16 to D12, D17 to D13, D15 to D14, D1 to D15, D2 to D16, D9 to D17, D7 to D18, D8 to D19, D4 to D2, D12 to D20, D10 to D21, D11 to D22, D18 to D3, D6 to D4, D21 to D5, D3 to D6, D13 to D7, D14 to D8, D5 to D9, J8 to J2, J6 to J3, J3 to J4, J4 to J5, J7 to J6, J2 to J7, J5 to J8, K2 to K1, K1 to K2, Q9 to Q1, Q4 to Q10, Q3 to Q2, Q10 to Q3, Q1 to Q4, Q11 to Q5, Q5 to Q6, Q6 to Q8, Q2 to Q9, R45 to R1, R33 to R10, R36 to R11, R46 to R12, R1 to R13, R2 to R14, R26 to R15, R27 to R16, R8 to R17, R30 to R18, R31 to R19, R7 to R2, R9 to R20, R32 to R21, R44 to R26, R10 to R27, R39 to R28, R40 to R29, R6 to R3, R41 to R30, R42 to R31, R43 to R32, R12 to R33, R14 to R34, R16 to R35, R18 to R36, R20 to R37, R21 to R38, R13 to R39, R11 to R4, R15 to R40, R17 to R41, R19 to R42, R3 to R5, R4 to R6, R28 to R7, R29 to R8, R5 to R9

Commit message: フットプリント割当、ERCOK
Parts:
- C1, C3, C4: footprint (none) -> Capacitor_SMD:C_0603_1608Metric
- C2: footprint (none) -> Capacitor_SMD:C_1206_3216Metric
- D10, D19, D3, D7, D8, D9: footprint (none) -> LED_SMD:LED_0603_1608Metric
- R1, R10, R11, R12, R13, R14, R15, R16, R17, R18, R19, R2, R20, R27, R3, R37, R38, R4, R5, R6, R7, R8, R9: footprint (none) -> Resistor_SMD:R_0603_1608Metric
